File: PSP4.sch (KiCad schematic (older format))
At the start: 63 parts

Commit message: more tweaking
Parts:
- added C? (x4): 22p, ~, symbol C_US
- added C? (x3): 100n, ~, symbol C_US
- added R? (x4): 10K, ~, symbol R_US
- added R? (x4): 68K, symbol R_US
- added R? (x4): 22K, symbol R_US
- added U? (x3): SN7407, symbol SN7407
- added U? (x4): OPA4171, symbol TL074-
- added U? (x3): CD4051, symbol CD4051
- added VR? (x4): 1K, symbol POT_US
Connections:
- net +12V: now also C?.1, C?.1, C?.1, R?.2, R?.2, R?.2, R?.2, U?.16 (VDD), U?.16 (VDD), U?.16 (VDD), U?.4 (V+)
- net -12V: now also U?.11 (V-)
- net CV1: now also C?.1, U?.14 (X1), U?.5 (+); no longer C?.1, U?.3 (+)
- net CV2: now also C?.1, U?.10 (+), U?.15 (X2); no longer C?.1, U?.5 (+)
- net CV3: now also C?.1, U?.12 (+), U?.12 (X3); no longer C?.1, U?.10 (+)
- net CV4: now also C?.1, U?.1 (X4), U?.3 (+); no longer C?.1, U?.12 (+)
- net CV5: now also C?.1, U?.5 (+), U?.5 (X5); no longer C?.1, U?.3 (+)
- net CV6: now also C?.1, U?.10 (+), U?.2 (X6); no longer C?.1, U?.5 (+)
- net CV7: now also C?.1, U?.12 (+), U?.4 (X7); no longer C?.1, U?.10 (+)
- net CV8: now also U?.13 (X0); no longer C?.1, U?.12 (+)
- net GND: now also C?.2, C?.2, C?.2, R?.2, R?.2, R?.2, R?.2, U?.7 (VEE), U?.7 (VEE), U?.7 (VEE), U?.8 (VSS), U?.8 (VSS), U?.8 (VSS)
- net at U?.11 (OUT2): now also U?.10 (+)
- net at U?.14 (OUT1): now also U?.5 (+)
- net at U?.3 (OUT0): now also U?.3 (+)
- net at U?.6 (OUT3): now also U?.12 (+)
- net B: now reaches U?.10 (B)
- net B: now also R?.1, U?.10 (B), U?.10 (B), U?.10 (B), U?.4
- net A: now reaches U?.11 (A)
- net A: now also U?.2, R?.1, U?.11 (A), U?.11 (A), U?.11 (A)
- net CV0: now reaches U?.13 (X0)
- net CV0: now also C?.1, U?.3 (+)
- net VDAC1: now reaches U?.3 (X)
- net VDAC1: now also C?.1, U?.1, VR?.2, VR?.3
- net ~DAC_MUX0_EN: now reaches U?.6 (Inh)
- net ~DAC_MUX0_EN: now also R?.1, U?.2
- net C: now reaches U?.9 (C)
- net C: now also R?.1, U?.6, U?.9 (C), U?.9 (C), U?.9 (C)
- net D0: now reaches U?.1
- new net: C?.2, R?.1, R?.2, U?.2 (-)
- new net: R?.1, VR?.1 (x4)
- new net: C?.2, R?.1, R?.2, U?.6 (-)
- new net: C?.2, R?.1, R?.2, U?.9 (-)
- new net: C?.2, R?.1, R?.2, U?.13 (-)
- new net CV10: U?.15 (X2)
- new net CV11: U?.12 (X3)
- new net CV12: U?.1 (X4)
- new net CV13: U?.5 (X5)
- new net CV14: U?.2 (X6)
- new net CV15: U?.4 (X7)
- new net CV16: U?.13 (X0)
- new net CV17: U?.14 (X1)
- new net CV18: U?.15 (X2)
- new net CV19: U?.12 (X3)
- new net CV20: U?.1 (X4)
- new net CV21: U?.5 (X5)
- new net CV22: U?.2 (X6)
- new net CV23: U?.4 (X7)
- new net CV24: U?.13 (X0)
- new net CV25: U?.14 (X1)
- new net CV26: U?.15 (X2)
- new net CV27: U?.12 (X3)
- new net CV28: U?.1 (X4)
- new net CV29: U?.5 (X5)
- new net CV30: U?.2 (X6)
- new net CV31: U?.4 (X7)
- new net CV9: U?.14 (X1)
- new net D1: U?.3
- new net D2: U?.5
- new net VDAC2: C?.1, U?.3 (X), U?.7, VR?.2, VR?.3
- new net VDAC3: C?.1, U?.3 (X), U?.8, VR?.2, VR?.3
- new net VDAC4: C?.1, U?.14, U?.3 (X), VR?.2, VR?.3
- new net ~DAC_MUX0: U?.1
- new net ~DAC_MUX1_EN: U?.6 (Inh)
- new net ~DAC_MUX2_EN: U?.6 (Inh)
- new net ~DAC_MUX3_EN: U?.6 (Inh)
Other:
- moved on the sheet: C?, R?, U?, U?A, U?B, U?C

Commit message: added envelopes to schematic
Parts:
- added C? (x2): 100p, MyModules:SM0603-C-JRL, symbol C_US
- added C? (x2): 100n**, MyModules:SM0603-C-JRL, symbol C_US
- added C? (x8): 100n, MyModules:SM0603-C-JRL, symbol C_US
- added Q? (x4): DMMT3904, MyModules:SOT363-JRL, symbol DMMT3904
- added Q? (x4): DMMT3906, MyModules:SOT363-JRL, symbol DMMT3906
- added Q? (x3): 2SC4738, SOT-23, symbol 2SC4738
- added R? (x2): 15K, MyModules:SM0603-R-JRL, symbol R_US
- added R? (x4): 82K*, MyModules:SM0603-R-JRL, symbol R_US
- added R? (x2): 150K, MyModules:SM0603-R-JRL, symbol R_US
- added R? (x9): 47K, MyModules:SM0603-R-JRL, symbol R_US
- added R? (x6): 2.2K, MyModules:SM0603-R-JRL, symbol R_US
- added R? (x2): 22K, MyModules:SM0603-R-JRL, symbol R_US
- added R? (x2): 33K, MyModules:SM0603-R-JRL, symbol R_US
- added R? (x5): 100K, MyModules:SM0603-R-JRL, symbol R_US
- added R? (x2): 330K, MyModules:SM0603-R-JRL, symbol R_US
- added R? (x3): 10K, MyModules:SM0603-R-JRL, symbol R_US
- added R? (x4): 270K, MyModules:SM0603-R-JRL, symbol R_US
- added R? (x2): 3.3K**, MyModules:SM0603-R-JRL, symbol R_US
- added R? (x4): 4.7K, MyModules:SM0603-R-JRL, symbol R_US
- added R?: 68K, MyModules:SM0603-R-JRL, symbol R_US
- added U? (x8): TL074-, Housings_SSOP:TSSOP-14_4.4x5mm_Pitch0.65mm, symbol TL074-
- added U? (x2): CD4052, Housings_SSOP:TSSOP-16_4.4x5mm_Pitch0.65mm, symbol CD4052
- added U? (x2): NE555, MyModules:TSSOP8-JRL, symbol NE555
Connections:
- net +12V: now also C?.1, C?.1, C?.1, C?.1, R?.1, R?.1, R?.1, R?.1, R?.2, R?.2, R?.2, R?.2, R?.2, U?.16 (VDD), U?.16 (VDD), U?.4 (R), U?.4 (R), U?.4 (V+), U?.4 (V+), U?.8 (VCC), U?.8 (VCC)
- net -12V: now also C?.2, C?.2, R?.1, R?.1, R?.1, R?.1, R?.2, R?.2, U?.11 (V-), U?.11 (V-)
- net GND: now also C?.1, C?.1, C?.2, C?.2, C?.2, C?.2, Q?.1, Q?.1, Q?.1, Q?.1, Q?.2 (E), Q?.2 (E), Q?.2 (E), R?.1, R?.1, R?.1, R?.1, R?.2, R?.2, R?.2, R?.2, U?.1 (GND), U?.1 (GND), U?.11 (X3), U?.11 (X3), U?.14 (X1), U?.14 (X1), U?.2 (Y2), U?.2 (Y2), U?.3 (+), U?.3 (+), U?.3 (+), U?.3 (+), U?.6 (Inh), U?.6 (Inh), U?.7 (VEE), U?.7 (VEE), U?.8 (VSS), U?.8 (VSS)
- new net: C?.1, R?.1, U?.1 (x2)
- new net: C?.2, Q?.6, Q?.6, R?.1, U?.2 (-) (x2)
- new net: C?.1, Q?.3 (C), R?.1, U?.10 (A) (x2)
- new net: R?.1, U?.13 (X) (x2)
- new net: R?.2, U?.15 (X2) (x2)
- new net: R?.1, U?.3 (Y) (x2)
- new net: U?.3 (Q), U?.9 (B) (x2)
- new net: R?.1, R?.2 (x4)
- new net: R?.1, R?.2, U?.1 (x2)
- new net: R?.1, R?.2, U?.2 (-) (x3)
- new net: R?.1, R?.2, U?.3 (+) (x2)
- new net: C?.1, R?.1, R?.1, R?.2, U?.1, U?.6 (THR)
- new net: C?.1, R?.2, U?.1, U?.3 (+), U?.6 (THR)
- new net: Q?.5, Q?.5, Q?.5, Q?.5, R?.2 (x2)
- new net: C?.2, Q?.6, Q?.6, U?.2 (-) (x2)
- new net: C?.2, R?.2, U?.2 (TR) (x2)
- new net: R?.1, U?.5 (CV) (x2)
- new net: Q?.1 (B), R?.1, R?.1 (x2)
- new net: Q?.1, R?.2, R?.2, R?.2 (x4)
- new net: R?.2, U?.3 (+)
- new net: Q?.3 (C), R?.1, R?.2
- new net: Q?.1 (B), R?.1
- new net ENV1_A: R?.1
- new net ENV1_D: U?.1 (Y0)
- new net ENV1_POL: R?.2
- new net ENV1_R: U?.4 (Y3), U?.5 (Y1)
- new net ENV1_S: U?.12 (X0)
- new net ENV2_A: R?.1
- new net ENV2_D: U?.1 (Y0)
- new net ENV2_R: U?.4 (Y3), U?.5 (Y1)
- new net ENV2_S: U?.12 (X0)
- new net ENV_1: R?.2, U?.1
- new net ENV_2: U?.1, U?.2 (-)
- new net GATE: R?.1, R?.1, R?.2, R?.2
- no-connect marks 4 -> 8
Other:
- note added: "**adust R to get \nthreshold of 10V"
- note added: "**match C5 value between\n ADSR modules. 95nF gives\nmin attack of <1.5ms"
- note added: "*\nADJUST R7/R8 with T1/T2 \nto get 20-25 s max A/D/R\n"
- note added: "+5V"
- note added: "0-10V CV"
- note added: "Change to PMP4201/5201 pairs?"
- note added: "ENV 1"
- note added: "ENV 2"
- note added: "ENV1 inversion works\nin simulation"
- note added: "R224A - omit?"
- note added: "VC ADSR"
- note added: "original design by Massimo Ischia\nhttp://digilander.libero.it/ismsynth/vc-adsr-1.2.jpg\nadapted for 0-10V input and 0-10V output"

Commit message: chipping away. finished off MAX5134 DAC schematic and sorted out DAC Vref and decoupling, working through level shifting switching signals
Parts:
- added C?: 100p, ~, symbol C_US
- added C?: 1μ, ~, symbol C_US
- added R?: 1K, ~, symbol R_US
- added R? (x7): 10K, ~, symbol R_US
- added U? (x7): SN7407, symbol SN7407
Connections:
- net +12V: now also R?.2, R?.2, R?.2, R?.2, R?.2, R?.2, R?.2
- net +5V: now also U?.14 (VCC)
- net GND: now also C?.2, U?.13 (M/~Z~), C?.2, C?.2, U?.7 (GND)
- net ~DAC_MUX0: now also U?.9; no longer U?.1
- net ~DAC_MUX0_EN: now also U?.8; no longer U?.2
- net ~DAC_MUX1_EN: now also R?.1, U?.10
- net ~DAC_MUX2_EN: now also R?.1, U?.12
- net at U?.1 (REFI): now also U?.16 (REF0), C?.1, R?.1
- net ~LDAC: now reaches U?.12 (~LDAC~)
- net ~DS0 renamed ~DAC_SEL
- new net: C?.1, R?.2
- new net DAC_MUX3: U?.1
- new net DAC_MUX3_EN: R?.1, U?.2
- new net VCO1_MOD_A: U?.3
- new net VCO1_MOD_A_SW: R?.1, U?.4
- new net VCO1_MOD_B: U?.5
- new net VCO1_MOD_B_SW: R?.1, U?.6
- new net VCO1_MOD_SOURCE_A: U?.9
- new net VCO1_MOD_SOURCE_A_SW: R?.1, U?.8
- new net VCO1_MOD_SOURCE_B: U?.11
- new net VCO1_MOD_SOURCE_B_SW: R?.1, U?.10
- new net ~DAC_MUX1: U?.11
- new net ~DAC_MUX2: U?.13
Other:
- moved on the sheet: C?

Commit message: label envelope CVs and switch signals"
a
dsfassa
Parts:
- added R? (x7): 10K, ~, symbol R_US
- added U? (x7): SN7407, symbol SN7407
Connections:
- net +12V: now also R?.2, R?.2, R?.2, R?.2, R?.2, R?.2, R?.2
- net +5V: now also U?.14 (VCC)
- net GND: now also U?.5 (+), U?.7 (GND); no longer U?.3 (+)
- net at R?.1, R?.2: now also U?.14; no longer U?.1
- net at R?.1, R?.2: now also U?.13 (-); no longer U?.2 (-)
- net at R?.1, R?.2: now also U?.12 (+); no longer U?.3 (+)
- net at C?.1, R?.1, R?.1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: now also U?.7; no longer U?.1
- net at C?.2, Q?.6, Q?.6: now also U?.6 (-); no longer U?.2 (-)
- net at R?.1, R?.2: now also U?.9 (-); no longer U?.2 (-)
- net at R?.2: now also U?.10 (+); no longer U?.3 (+)
- net ENV1_A renamed ATTACK_2A
- net ENV1_D renamed DECAY_2A
- net ENV1_POL renamed EG2_POL_A_SW
- net EG2_POL_A_SW: now also R?.1, U?.4
- net ENV1_R renamed RELEASE_2A
- net ENV1_S renamed SUSTAIN_2A
- net ENV2_A renamed ATTACK_1A
- net ENV2_D renamed DECAY_1A
- net ENV2_R renamed RELEASE_1A
- net ENV2_S renamed SUSTAIN_1A
- net ENV_1 renamed EG2_A
- net EG2_A: now also U?.8; no longer U?.1
- net ENV_2 renamed EG1_A
- net GATE renamed GATE_A
- new net: R?.1, U?.8
- new net: R?.1, U?.10
- new net: R?.1, U?.12
- new net EG2_POL_A: U?.3
- new net EG2_POL_B: U?.5
- new net EG2_POL_B_SW: R?.1, U?.6
- new net LFO_MODE_A: U?.13
- new net LFO_MODE_A_SW: R?.1, U?.12
- new net LFO_MODE_B: U?.1
- new net LFO_MODE_B_SW: R?.1, U?.2
Other:
- note added: "ENV1 A"
- note added: "ENV2 A"
- note removed: "ENV 1"
- note removed: "ENV 2"
- note removed: "VC ADSR"
- note removed: "original design by Massimo Ischia\nhttp://digilander.libero.it/ismsynth/vc-adsr-1.2.jpg\nadapted for 0-10V input and 0-10V output"
- moved on the sheet: C?, Q?, Q?A, R?, U?, U?A, U?B, U?C, U?D, U?E, U?F

Commit message: four envelope schematics now in hierarchical sheets
Parts:
- removed C? (x2): 100p, MyModules:SM0603-C-JRL, symbol C_US
- removed C? (x2): 100n**, MyModules:SM0603-C-JRL, symbol C_US
- removed C? (x8): 100n, MyModules:SM0603-C-JRL, symbol C_US
- removed Q? (x4): DMMT3904, MyModules:SOT363-JRL, symbol DMMT3904
- removed Q? (x4): DMMT3906, MyModules:SOT363-JRL, symbol DMMT3906
- removed Q? (x3): 2SC4738, SOT-23, symbol 2SC4738
- removed R? (x2): 15K, MyModules:SM0603-R-JRL, symbol R_US
- removed R? (x4): 82K*, MyModules:SM0603-R-JRL, symbol R_US
- removed R? (x2): 150K, MyModules:SM0603-R-JRL, symbol R_US
- removed R? (x9): 47K, MyModules:SM0603-R-JRL, symbol R_US
- removed R? (x6): 2.2K, MyModules:SM0603-R-JRL, symbol R_US
- removed R? (x2): 22K, MyModules:SM0603-R-JRL, symbol R_US
- removed R? (x2): 33K, MyModules:SM0603-R-JRL, symbol R_US
- removed R? (x5): 100K, MyModules:SM0603-R-JRL, symbol R_US
- removed R? (x2): 330K, MyModules:SM0603-R-JRL, symbol R_US
- removed R? (x3): 10K, MyModules:SM0603-R-JRL, symbol R_US
- removed R? (x4): 270K, MyModules:SM0603-R-JRL, symbol R_US
- removed R? (x2): 3.3K**, MyModules:SM0603-R-JRL, symbol R_US
- removed R? (x4): 4.7K, MyModules:SM0603-R-JRL, symbol R_US
- removed R?: 68K, MyModules:SM0603-R-JRL, symbol R_US
- removed U? (x8): TL074-, Housings_SSOP:TSSOP-14_4.4x5mm_Pitch0.65mm, symbol TL074-
- removed U? (x2): CD4052, Housings_SSOP:TSSOP-16_4.4x5mm_Pitch0.65mm, symbol CD4052
- removed U? (x2): NE555, MyModules:TSSOP8-JRL, symbol NE555
Connections:
- no-connect marks 8 -> 5
Other:
- note added: "PORTAMENTO A\n"
- note added: "PORTAMENTO B\n"
- note removed: "**adust R to get \nthreshold of 10V"
- note removed: "**match C5 value between\n ADSR modules. 95nF gives\nmin attack of <1.5ms"
- note removed: "*\nADJUST R7/R8 with T1/T2 \nto get 20-25 s max A/D/R\n"
- note removed: "+5V"
- note removed: "0-10V CV"
- note removed: "ADAPTED FROM SCI PROPHET 5 GLIDE CIRCUIT"
- note removed: "Change to PMP4201/5201 pairs?"
- note removed: "ENV1 A"
- note removed: "ENV1 inversion works\nin simulation"
- note removed: "ENV2 A"
- note removed: "GLIDE A\n"
- note removed: "GLIDE B\n"
- note removed: "R224A - omit?"
- moved on the sheet: R?, U?A, U?B, U?C, U?D, U?E, U?F
